Commit message: update sake

File: urdf/sake.urdf (robot description, URDF)
Before this commit: robot multishapes, 3 links, 2 joints
Links:
- added link arm_rotator_link; visual box size=0.03 0.03 0.03
- link base_link: geometry visual cylinder length=0.1 radius=0.05
- link base_rotator_link: geometry visual sphere radius=0.05
- link link_arm: geometry visual cylinder length=0.3 radius=0.013
Joints:
- added joint base_arm_to_arm_rotator_joint: type continuous, parent link_arm, child arm_rotator_link, axis 1 1 0.2
- joint base_arm_joint: axis (none) -> 1 0 0; origin xyz=0 0.1 0.3  rpy=0 0 0 -> xyz=0 0 0  rpy=0 1 0
- joint base_to_rotoator_joint: axis 0 0 1 -> 0 0 0.1; origin xyz=0 0 0.04 -> xyz=0 0 0.1 rpy=0 0 0
